File: Sodimm-force.kicad_pcb (KiCad board)
At the start: 8 copper layers, 67.6 x 25.4 mm, 186 parts, among them J1 SODIMM-200_Split, J2 HDMI_C_1.4, J3 Micro_SD_Card_Det2, J4 USB_C_Receptacle_USB2.0_16P, J5 USB_C_Receptacle_USB2.0_16P, Q1 2N7002, SW1 SW_Push, SW2 SW_Push, SW3 SW_Push, SW4 SW_Push, U1 SPX3819M5-L, U2 SPX3819M5-L, U3 SPI-EEPROM, Y1 X322524MKB4SI

Commit message: DDR оттрассирована!! 🥹
Parts:
- moved J1 72.3 mm to (98.0, 152.4)
- moved DD1 35.8 mm to (124.1, 134.9)
- moved DD6 35.8 mm to (137.1, 138.6)
Routing:
- net VCC-DRAM: track 0.00 -> 51.7 mm, vias 6 -> 29
- net Earth: track 0.07 -> 36.6 mm, vias 26 -> 53
- net SDQS0P: track 13.1 -> 34.8 mm
- net SDQS0N: track 13.7 -> 35.3 mm
- net SDQ8: track 14.7 -> 35.2 mm
- net SDQ11: track 15.2 -> 35.6 mm
- net SDQ14: track 15.5 -> 35.7 mm
- net SDQ13: track 16.9 -> 35.6 mm
- net SDQ10: track 17.1 -> 35.2 mm
- net SDQ12: track 17.0 -> 34.0 mm
- net SDQ9: track 18.9 -> 35.8 mm
- net SA1: track 23.2 -> 38.2 mm
- net SDQM1: track 21.3 -> 35.3 mm
- net SA0: track 24.9 -> 38.7 mm
- net SCS0: track 33.8 -> 46.5 mm
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- added copper zone on F.Cu, net Earth
- added copper zone on F.Cu, net VCC-DRAM
Other:
- outline, holes or cut-outs redrawn
