File: HDMI + usb.kicad_sch (KiCad schematic)
At the start: 49 parts, among them Q1 2N7002, SW1 SW_Push, SW2 SW_Push, SW3 SW_Push, SW4 SW_Push, U3 M24M02-DRMN6TP, X2 HDMI_C_1.4, X3 Micro_SD_Card_Det2, X4 USB_C_Receptacle_USB2.0_16P, X5 USB_C_Receptacle_USB2.0_16P

Commit message: GOST update
Parts:
- renumbered U3 to DD7
Other:
- moved on the sheet: D3
Changed lines of the file:
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@@
 	(wire
 		(pts
-			(xy 285.75 163.83) (xy 285.75 162.56)
+			(xy 284.48 163.83) (xy 284.48 162.56)
 		)
 		(stroke
@@
 	(wire
 		(pts
-			(xy 292.1 142.24) (xy 285.75 142.24)
+			(xy 292.1 142.24) (xy 284.48 142.24)
 		)
 		(stroke
@@
 		(on_board yes)
 		(dnp no)
-		(property "Reference" "U3"
+		(property "Reference" "DD7"
 			(at 91.694 134.874 0)
 			(effects
@@
 			(project "Sodimm-force"
 				(path "/b3673bfd-24d8-4789-b63c-c3654dc2bb6e/526c7efe-cb70-49a2-a6ca-c3db3e12ecbe"
-					(reference "U3")
+					(reference "DD7")
 					(unit 1)
 				)
@@
 		)
 		(property "Value" "10K"
-			(at 114.554 63.246 0)
+			(at 114.3 63.246 0)
 			(effects
 				(font
@@
 	(symbol
 		(lib_id "power:Earth")
-		(at 285.75 163.83 0)
+		(at 284.48 163.83 0)
 		(mirror y)
 		(unit 1)
@@
 		(fields_autoplaced yes)
 		(property "Reference" "#PWR0178"
-			(at 285.75 170.18 0)
+			(at 284.48 170.18 0)
 			(effects
 				(font
@@
 		)
 		(property "Value" "Earth"
-			(at 285.75 168.91 0)
+			(at 284.48 168.91 0)
 			(effects
 				(font
@@
 		)
 		(property "Footprint" ""
-			(at 285.75 163.83 0)
+			(at 284.48 163.83 0)
 			(effects
 				(font
@@
 		)
 		(property "Datasheet" "~"
-			(at 285.75 163.83 0)
+			(at 284.48 163.83 0)
 			(effects
 				(font
@@
 		)
 		(property "Description" "Power symbol creates a global label with name \"Earth\""
-			(at 285.75 163.83 0)
+			(at 284.48 163.83 0)
 			(effects
 				(font
@@
 		(dnp no)
 		(property "Reference" "R36"
-			(at 109.474 61.722 0)
+			(at 109.22 61.722 0)
 			(effects
 				(font
@@
 		)
 		(property "Value" "10K"
-			(at 109.474 63.246 0)
+			(at 109.22 63.246 0)
 			(effects
 				(font
@@
 		)
 		(property "Value" "VDD33"
-			(at 307.594 232.41 0)
+			(at 306.324 232.41 90)
 			(effects
 				(font
+					(face "GOST type A")
 					(size 1.27 1.27)
 				)
@@
 	(symbol
 		(lib_id "ESD:AZ5825-01F")
-		(at 285.75 142.24 90)
+		(at 284.48 142.24 90)
 		(mirror x)
 		(unit 1)
@@
 		(dnp no)
 		(property "Reference" "D3"
-			(at 282.448 149.86 90)
+			(at 281.178 149.86 90)
 			(effects
 				(font
@@
 		)
 		(property "Value" "AZ5825-01F"
-			(at 279.908 154.178 90)
+			(at 278.638 154.178 90)
 			(effects
 				(font
@@
 		)
 		(property "Footprint" "ESD:AZ582501F"
-			(at 379.4 154.94 0)
+			(at 378.13 154.94 0)
 			(effects
 				(font
@@
 		)
 		(property "Datasheet" ""
-			(at 381 138.684 0)
+			(at 379.73 138.684 0)
 			(effects
 				(font
@@
 		)
 		(property "Description" ""
-			(at 289.306 143.51 0)
+			(at 288.036 143.51 0)
 			(effects
 				(font
@@
 		)
 		(property "Height" " "
-			(at 679.4 154.94 0)
+			(at 678.13 154.94 0)
 			(effects
 				(font
@@
 		)
 		(property "Manufacturer_Name" " "
-			(at 779.4 154.94 0)
+			(at 778.13 154.94 0)
 			(effects
 				(font
@@
 		)
 		(property "Manufacturer_Part_Number" " "
-			(at 879.4 154.94 0)
+			(at 878.13 154.94 0)
 			(effects
 				(font
@@
 		)
 		(property "Mouser Part Number" " "
-			(at 979.4 154.94 0)
+			(at 978.13 154.94 0)
 			(effects
 				(font
@@
 		)
 		(property "Mouser Price/Stock" " "
-			(at 1079.4 154.94 0)
+			(at 1078.13 154.94 0)
 			(effects
 				(font
@@
 		)
 		(property "Arrow Part Number" " "
-			(at 1179.4 154.94 0)
+			(at 1178.13 154.94 0)
 			(effects
 				(font
@@
 		)
 		(property "Arrow Price/Stock" ""
-			(at 1279.4 154.94 0)
+			(at 1278.13 154.94 0)
 			(effects
 				(font
