File: power.kicad_sch (KiCad schematic)
At the start: 51 parts, among them U1 SPX3819M5-L, U2 SPX3819M5-L

Commit message: Исправление УГО по ГОСТу, добавление 3D моделей
Parts:
- DD1: value ~ -> H616
Other:
- company: @madjogger -> РТУ МИРЭА

Commit message: GOST update
Parts:
- renumbered U1 to DA1, U2 to DA2
Changed lines of the file:
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@@
 			"AAAAAAAAAAAAAAAAAAAAAAAAAAAAAAAAAAAAAAAAAAAAAAAAAAAAAAAAAAAAAAAAAAAAAAAAAAAA"
 			"AAAAAAAAAAAAAAAAAAAAAAAAAAAAAAAAAAAAAAAAAAAAfZhK5gBHAIABAAAAAAAAAMDZnU5gAgAA"
-			"AgAAAA=="
+			"AgAAAEsAWAB0ADIAbQBjAC8AQgBuADIAOQBnAFEAbQBUAEgAaQBIAE0AZgBWAFQATwBQAFQANwBR"
+			"AGMANwAvAHcAMwBxADEAQgArADUAbgArAG0AbQBPAG4AVQBtAGoAawBsAC8AOQBYAEwATgBiAEYA"
+			"bgBYAHIAVQBzAE0AMABuAG8AaAB6AHMAVwBEAGQAaABpADUAdAB5ADMARgA2ADYAeQArAEUANgAx"
+			"AFAAWgA5ACsAcwB1AE4ATwAzAGYAWQBXAHkATABWAFAANwBjADgAaQBkADMARABOAGYAWQB0AHUA"
+			"MABJADEAdQAyADYAMABLADYAcwBqAG4ATgBoADUAMABoAEoATwA4AFMAYwBQAGcARQBFAEIARwBS"
+			"ADgAZwB0ADcAZgB6AGkAMQBEAFAASABGAHgAVwBYACsANwBDAGUAVwBhAHQASwBOAEYAOABSADUA"
+			"UwBxAEMAaQBLAG8AaQBpAEsAOABsAEMAcABRAFoATAB5AEMASwBWAHcAWQBPADkAUgBVAGkAMgBy"
+			"ADQAKwB1AGQAKwAzADQAZgBnAEgASQBOAEcAbABMADkAMwBpACsAOAAyAHIAUQBoAEEAWQBFAHQA"
+			"YQBSAHkAOABHAHAAdABoADcAegBQAEMATgA1ADkAcABtAFEAZABJADIAZgBjAEIAZwBTADIASABN"
+			"AEQALwBDAGsAYQBiAGQAQgBqAEIAawBjAEcAZABxADIAZQBZAGQAZABPAFQATAB2AEIAbwAxAFAA"
+			"YwAxAEkAUAByAHkAWABJADUAbQB6AE0AaABhAFYAbQA5AE8AdABaAHkAOQA2ADkAUQB5AGsAbABr"
+			"AFAAZQBjAGsAeAByAGoAVwBmAEgAbABUAGoAaQBrACsANgBTAEcATABtAGIASgBlAFAAOABNADIA"
+			"ZQBoADgAdABLADQAVgBhAEsAaQBtAFkANgBMADQAZQBmAFEARwBXAC8ARQBRAE8AegBwAHMAOABU"
+			"AGgAUwBmAFgAcQB4AG4AKwB2AE8AZABWAHEAZQBtAEsAVwBmAEoAaQA5ADkAMwBlAE0ANQB0ADEA"
+			"NgAwAHEAdABYAFQAdwBKAHIATwBaAEIAMwB6ADMASgA3ADgASAA2AG0AawBaAFkAdQBhAEUAeQBO"
+			"AGgAbgBVAGEARABaAHIATQB4ADQAYQBDAEwAZQAyADcAdABNAGIAcQB4AEQAYQAyAG4ARAAvAEMA"
+			"cgAzADgAbQAwAGoAaQBnAEcAMQAwAEQANgA1AEgAdwArAHgAYgAyAHgAdgA3AEsAMQB2ADMAbQB0"
+			"AE8ANwA2AEQATABZAEkATwBwADAAZQB5AHQAVwBpAHkAKwBCAGgARABCAHUAVwArAFgAbgBsAEEA"
+			"KwBiAA=="
 		)
 	)
@@
 		(length 2.54)
 		(shape round)
-		(at 140.97 226.06 0)
+		(at 139.7 226.06 0)
 		(fields_autoplaced yes)
 		(effects
@@
 		)
 		(property "Netclass" "Power"
-			(at 141.6685 223.52 0)
+			(at 140.3985 223.52 0)
 			(effects
 				(font
@@
 		)
 		(property "Component Class" ""
-			(at 106.68 48.26 0)
+			(at 105.41 48.26 0)
 			(effects
 				(font
@@
 		(on_board yes)
 		(dnp no)
-		(property "Reference" "U2"
+		(property "Reference" "DA2"
 			(at 273.304 228.092 0)
 			(effects
@@
 			(project "Sodimm-force"
 				(path "/b3673bfd-24d8-4789-b63c-c3654dc2bb6e/80cb261a-71dc-4751-a2b6-2fe7421285af"
-					(reference "U2")
+					(reference "DA2")
 					(unit 1)
 				)
@@
 		(on_board yes)
 		(dnp no)
-		(property "Reference" "U1"
+		(property "Reference" "DA1"
 			(at 273.304 192.532 0)
 			(effects
@@
 			(project ""
 				(path "/b3673bfd-24d8-4789-b63c-c3654dc2bb6e/80cb261a-71dc-4751-a2b6-2fe7421285af"
-					(reference "U1")
+					(reference "DA1")
 					(unit 1)
 				)
